File: keyboard/keyboard.kicad_sch (KiCad schematic)
At the start: 168 parts, among them J1 Conn_01x20_Pin, SW1 SW_Push, SW2 SW_Push

Commit message: Add files via upload
Parts:
- removed J1: Conn_01x20_Pin, symbol Connector:Conn_01x20_Pin
- removed SW2: SW_Push, symbol Switch:SW_Push
- added D100, D101, D102, D103, D104, D105, D106, D107, D108, D109, D110, D111, D112, D113, D114, D115, D116, D117, D118, D119, D120, D121, D122, D123, D124, D125, D126, D127, D128, D129, D130, D131, D132, D133, D134, D135, D136, D137, D138, D139, D140, D141, D142, D143, D144, D145, D146, D147, D148, D149, D150, D151, D152, D153, D154, D155, D156, D76, D80, D81, D82, D83, D84, D85, D86, D87, D88, D89, D90, D91, D92, D93, D94, D95, D96, D97, D98, D99: SK6812MINI-E, LED_SMD:LED_SK6812MINI-E_3.2x2.8mm_P1.5mm_ReverseMount, symbol LED:SK6812MINI-E
- added D157, D158, D159, D160, D161: D, Diode_THT:D_DO-35_SOD27_P7.62mm_Horizontal, symbol Device:D
- added EC3, EC4, EC5: RotaryEncoder_Switch, Rotary_Encoder:RotaryEncoder_Alps_EC11E-Switch_Vertical_H20mm, symbol Device:RotaryEncoder_Switch
- added J1: Conn_01x14_Pin, Connector_PinHeader_2.54mm:PinHeader_1x14_P2.54mm_Vertical, symbol Connector:Conn_01x14_Pin
- added J3: Conn_01x06_Pin, Connector_PinHeader_2.54mm:PinHeader_1x06_P2.54mm_Vertical, symbol Connector:Conn_01x06_Pin
- added J4, J5: Conn_01x02_Pin, Connector_PinHeader_2.54mm:PinHeader_1x02_P2.54mm_Vertical, symbol Connector:Conn_01x02_Pin
- added LEDDEBUG1: SW_Push, PTS810_SJM_250_SMTR_LFS:SW_PTS810_SJM_250_SMTR_LFS, symbol Switch:SW_Push
- added R10, R11, R12, R9: 10k, Resistor_SMD:R_0805_2012Metric_Pad1.20x1.40mm_HandSolder, symbol Device:R
- A1, A2: footprint Module:RaspberryPi_Pico_SMD -> Module:RaspberryPi_Pico_Common_THT
- D1, D10, D11, D12, D13, D14, D15, D16, D17, D18, D19, D2, D20, D21, D22, D23, D24, D25, D26, D27, D28, D29, D3, D30, D31, D32, D33, D34, D35, D36, D37, D38, D39, D4, D40, D41, D42, D43, D44, D45, D46, D47, D48, D49, D5, D50, D51, D52, D53, D54, D55, D56, D57, D58, D59, D6, D60, D61, D62, D63, D64, D65, D66, D67, D68, D69, D7, D70, D71, D72, D73, D74, D75, D77, D78, D79, D8, D9: footprint (none) -> Diode_THT:D_DO-35_SOD27_P7.62mm_Horizontal
- DEBUG1: renamed from SW1; footprint (none) -> PTS810_SJM_250_SMTR_LFS:SW_PTS810_SJM_250_SMTR_LFS
- R1, R2, R3, R4, R6, R7: footprint (none) -> Resistor_SMD:R_0805_2012Metric_Pad1.20x1.40mm_HandSolder
- R5: value 4.7k -> 10k; footprint (none) -> Resistor_SMD:R_0805_2012Metric_Pad1.20x1.40mm_HandSolder
- SW1: renamed from Esc; footprint (none) -> Button_Switch_Keyboard:SW_Cherry_MX_1.00u_PCB
- SW10: renamed from F9; footprint (none) -> Button_Switch_Keyboard:SW_Cherry_MX_1.00u_PCB
- SW11: renamed from F10; footprint (none) -> Button_Switch_Keyboard:SW_Cherry_MX_1.00u_PCB
- SW12: renamed from F11; footprint (none) -> Button_Switch_Keyboard:SW_Cherry_MX_1.00u_PCB
- SW13: renamed from F12; footprint (none) -> Button_Switch_Keyboard:SW_Cherry_MX_1.00u_PCB
- SW14: renamed from `; footprint (none) -> Button_Switch_Keyboard:SW_Cherry_MX_1.00u_PCB
- SW15: renamed from _1; footprint (none) -> Button_Switch_Keyboard:SW_Cherry_MX_1.00u_PCB
- SW16: renamed from _2; footprint (none) -> Button_Switch_Keyboard:SW_Cherry_MX_1.00u_PCB
- SW17: renamed from _3; footprint (none) -> Button_Switch_Keyboard:SW_Cherry_MX_1.00u_PCB
- SW18: renamed from _4; footprint (none) -> Button_Switch_Keyboard:SW_Cherry_MX_1.00u_PCB
- SW19: renamed from _5; footprint (none) -> Button_Switch_Keyboard:SW_Cherry_MX_1.00u_PCB
- SW2: renamed from F1; footprint (none) -> Button_Switch_Keyboard:SW_Cherry_MX_1.00u_PCB
- SW20: renamed from _6; footprint (none) -> Button_Switch_Keyboard:SW_Cherry_MX_1.00u_PCB
- SW21: renamed from _7; footprint (none) -> Button_Switch_Keyboard:SW_Cherry_MX_1.00u_PCB
- SW22: renamed from _8; footprint (none) -> Button_Switch_Keyboard:SW_Cherry_MX_1.00u_PCB
- SW23: renamed from _9; footprint (none) -> Button_Switch_Keyboard:SW_Cherry_MX_1.00u_PCB
- SW24: renamed from _10; footprint (none) -> Button_Switch_Keyboard:SW_Cherry_MX_1.00u_PCB
- SW25: renamed from -; footprint (none) -> Button_Switch_Keyboard:SW_Cherry_MX_1.00u_PCB
- SW26: renamed from +; footprint (none) -> Button_Switch_Keyboard:SW_Cherry_MX_1.00u_PCB
- SW27: renamed from Backspace; footprint (none) -> Button_Switch_Keyboard:SW_Cherry_MX_2.00u_PCB
- SW28: renamed from Tab; footprint (none) -> Button_Switch_Keyboard:SW_Cherry_MX_1.50u_PCB
- SW29: renamed from q; footprint (none) -> Button_Switch_Keyboard:SW_Cherry_MX_1.00u_PCB
- SW3: renamed from F2; footprint (none) -> Button_Switch_Keyboard:SW_Cherry_MX_1.00u_PCB
- SW30: renamed from w; footprint (none) -> Button_Switch_Keyboard:SW_Cherry_MX_1.00u_PCB
- SW31: renamed from e; footprint (none) -> Button_Switch_Keyboard:SW_Cherry_MX_1.00u_PCB
- SW32: renamed from r; footprint (none) -> Button_Switch_Keyboard:SW_Cherry_MX_1.00u_PCB
- SW33: renamed from t; footprint (none) -> Button_Switch_Keyboard:SW_Cherry_MX_1.00u_PCB
- SW34: renamed from y; footprint (none) -> Button_Switch_Keyboard:SW_Cherry_MX_1.00u_PCB
- SW35: renamed from u; footprint (none) -> Button_Switch_Keyboard:SW_Cherry_MX_1.00u_PCB
- SW36: renamed from i; footprint (none) -> Button_Switch_Keyboard:SW_Cherry_MX_1.00u_PCB
- SW37: renamed from o; footprint (none) -> Button_Switch_Keyboard:SW_Cherry_MX_1.00u_PCB
- SW38: renamed from p; footprint (none) -> Button_Switch_Keyboard:SW_Cherry_MX_1.00u_PCB
- SW39: renamed from [; footprint (none) -> Button_Switch_Keyboard:SW_Cherry_MX_1.00u_PCB
- SW4: renamed from F3; footprint (none) -> Button_Switch_Keyboard:SW_Cherry_MX_1.00u_PCB
- SW40: renamed from ]; footprint (none) -> Button_Switch_Keyboard:SW_Cherry_MX_1.00u_PCB
- SW41: renamed from \; footprint (none) -> Button_Switch_Keyboard:SW_Cherry_MX_1.50u_PCB
- SW42: renamed from Caps; footprint (none) -> Button_Switch_Keyboard:SW_Cherry_MX_1.50u_PCB
- SW43: renamed from a; footprint (none) -> Button_Switch_Keyboard:SW_Cherry_MX_1.00u_PCB
- SW44: renamed from s; footprint (none) -> Button_Switch_Keyboard:SW_Cherry_MX_1.00u_PCB
- SW45: renamed from d; footprint (none) -> Button_Switch_Keyboard:SW_Cherry_MX_1.00u_PCB
- SW46: renamed from f; footprint (none) -> Button_Switch_Keyboard:SW_Cherry_MX_1.00u_PCB
- SW47: renamed from g; footprint (none) -> Button_Switch_Keyboard:SW_Cherry_MX_1.00u_PCB
- SW48: renamed from h; footprint (none) -> Button_Switch_Keyboard:SW_Cherry_MX_1.00u_PCB
- SW49: renamed from j; footprint (none) -> Button_Switch_Keyboard:SW_Cherry_MX_1.00u_PCB
- SW5: renamed from F4; footprint (none) -> Button_Switch_Keyboard:SW_Cherry_MX_1.00u_PCB
- SW50: renamed from k; footprint (none) -> Button_Switch_Keyboard:SW_Cherry_MX_1.00u_PCB
- SW51: renamed from l; footprint (none) -> Button_Switch_Keyboard:SW_Cherry_MX_1.00u_PCB
- SW52: renamed from ;; footprint (none) -> Button_Switch_Keyboard:SW_Cherry_MX_1.00u_PCB
- SW53: renamed from '; footprint (none) -> Button_Switch_Keyboard:SW_Cherry_MX_1.00u_PCB
- SW54: renamed from enter; footprint (none) -> Button_Switch_Keyboard:SW_Cherry_MX_2.25u_PCB
- SW55: renamed from Shift; footprint (none) -> Button_Switch_Keyboard:SW_Cherry_MX_2.25u_PCB
- SW56: renamed from z; footprint (none) -> Button_Switch_Keyboard:SW_Cherry_MX_1.00u_PCB
- SW57: renamed from x; footprint (none) -> Button_Switch_Keyboard:SW_Cherry_MX_1.00u_PCB
- SW58: renamed from c; footprint (none) -> Button_Switch_Keyboard:SW_Cherry_MX_1.00u_PCB
- SW59: renamed from v; footprint (none) -> Button_Switch_Keyboard:SW_Cherry_MX_1.00u_PCB
- SW6: renamed from F5; footprint (none) -> Button_Switch_Keyboard:SW_Cherry_MX_1.00u_PCB
- SW60: renamed from b; footprint (none) -> Button_Switch_Keyboard:SW_Cherry_MX_1.00u_PCB
- SW61: renamed from n; footprint (none) -> Button_Switch_Keyboard:SW_Cherry_MX_1.00u_PCB
- SW62: renamed from m; footprint (none) -> Button_Switch_Keyboard:SW_Cherry_MX_1.00u_PCB
- SW63: renamed from ,; footprint (none) -> Button_Switch_Keyboard:SW_Cherry_MX_1.00u_PCB
- SW64: renamed from .; footprint (none) -> Button_Switch_Keyboard:SW_Cherry_MX_1.00u_PCB
- SW65: renamed from /; footprint (none) -> Button_Switch_Keyboard:SW_Cherry_MX_1.00u_PCB
- SW66: renamed from shift; footprint (none) -> Button_Switch_Keyboard:SW_Cherry_MX_2.75u_PCB
- SW67: renamed from up; footprint (none) -> Button_Switch_Keyboard:SW_Cherry_MX_1.00u_PCB
- SW68, SW75: renamed from Ctrl; footprint (none) -> Button_Switch_Keyboard:SW_Cherry_MX_1.25u_PCB
- SW69: renamed from Win; footprint (none) -> Button_Switch_Keyboard:SW_Cherry_MX_1.25u_PCB
- SW7: renamed from F6; footprint (none) -> Button_Switch_Keyboard:SW_Cherry_MX_1.00u_PCB
- SW70: renamed from Alt; footprint (none) -> Button_Switch_Keyboard:SW_Cherry_MX_1.25u_PCB
- SW71: renamed from Space; footprint (none) -> Button_Switch_Keyboard:SW_Cherry_MX_6.25u_PCB
- SW72: renamed from alt; footprint (none) -> Button_Switch_Keyboard:SW_Cherry_MX_1.25u_PCB
- SW73: renamed from fn; footprint (none) -> Button_Switch_Keyboard:SW_Cherry_MX_1.25u_PCB
- SW74: renamed from smth; footprint (none) -> Button_Switch_Keyboard:SW_Cherry_MX_1.25u_PCB
- SW76: renamed from left; footprint (none) -> Button_Switch_Keyboard:SW_Cherry_MX_1.00u_PCB
- SW77: renamed from down; footprint (none) -> Button_Switch_Keyboard:SW_Cherry_MX_1.00u_PCB
- SW78: renamed from right; footprint (none) -> Button_Switch_Keyboard:SW_Cherry_MX_1.00u_PCB
- SW8: renamed from F7; footprint (none) -> Button_Switch_Keyboard:SW_Cherry_MX_1.00u_PCB
- SW9: renamed from F8; footprint (none) -> Button_Switch_Keyboard:SW_Cherry_MX_1.00u_PCB
Connections:
- net CD is gone; now on net SLAVEPWR: R2.2
- net CLK: now also J1.8 (Pin_8)
- net COL0: now also A1.11 (GPIO8)
- net COL1: now also A1.12 (GPIO9)
- net COL10: now also A1.26 (GPIO20)
- net COL11: now also A1.25 (GPIO19)
- net COL12: now also A1.24 (GPIO18)
- net COL13: now also A1.22 (GPIO17), EC3.S2, EC4.S2, EC5.S2
- net COL2: now also A1.14 (GPIO10)
- net COL3: now also A1.15 (GPIO11)
- net COL4: now also A1.16 (GPIO12)
- net COL5: now also A1.17 (GPIO13)
- net COL6: now also A1.19 (GPIO14)
- net COL7: now also A1.20 (GPIO15)
- net COL8: now also A1.29 (GPIO22)
- net COL9: now also A1.27 (GPIO21)
- net CS: now also R2.1, J1.12 (Pin_12); no longer R1.1
- net DC: now also A2.27 (GPIO21), J1.10 (Pin_10); no longer A2.29 (GPIO22)
- net GND: now also D100.1 (VSS), D101.1 (VSS), D102.1 (VSS), D103.1 (VSS), D104.1 (VSS), D105.1 (VSS), D106.1 (VSS), D107.1 (VSS), D108.1 (VSS), D109.1 (VSS), D110.1 (VSS), D111.1 (VSS), D112.1 (VSS), D113.1 (VSS), D114.1 (VSS), D115.1 (VSS), D116.1 (VSS), D117.1 (VSS), D118.1 (VSS), D119.1 (VSS), D120.1 (VSS), D121.1 (VSS), D122.1 (VSS), D123.1 (VSS), D124.1 (VSS), D125.1 (VSS), D126.1 (VSS), D127.1 (VSS), D128.1 (VSS), D129.1 (VSS), D130.1 (VSS), D131.1 (VSS), D132.1 (VSS), D133.1 (VSS), D134.1 (VSS), D135.1 (VSS), D136.1 (VSS), D137.1 (VSS), D138.1 (VSS), D139.1 (VSS), D140.1 (VSS), D141.1 (VSS), D142.1 (VSS), D143.1 (VSS), D144.1 (VSS), D145.1 (VSS), D146.1 (VSS), D147.1 (VSS), D148.1 (VSS), D149.1 (VSS), D150.1 (VSS), D151.1 (VSS), D152.1 (VSS), D153.1 (VSS), D154.1 (VSS), D155.1 (VSS), D156.1 (VSS), D76.1 (VSS), D80.1 (VSS), D81.1 (VSS), D82.1 (VSS), D83.1 (VSS), D84.1 (VSS), D85.1 (VSS), D86.1 (VSS), D87.1 (VSS), D88.1 (VSS), D89.1 (VSS), D90.1 (VSS), D91.1 (VSS), D92.1 (VSS), D93.1 (VSS), D94.1 (VSS), D95.1 (VSS), D96.1 (VSS), D97.1 (VSS), D98.1 (VSS), D99.1 (VSS), EC3.C, EC4.C, EC5.C, J1.13 (Pin_13), J3.3 (Pin_3), J4.1 (Pin_1), J5.1 (Pin_1), LEDDEBUG1.1; no longer R7.2
- net MISO: now also J1.6 (Pin_6)
- net MOSI: now also J1.9 (Pin_9)
- net ROW0: now also A1.4 (GPIO2), D158.1 (K)
- net ROW1: now also A1.5 (GPIO3)
- net ROW2: now also A1.6 (GPIO4)
- net ROW3: now also A1.7 (GPIO5), D159.1 (K)
- net ROW4: now also A1.9 (GPIO6), D160.1 (K)
- net ROW5: now also A1.10 (GPIO7)
- net RUN: now also D157.1 (K), D161.1 (K); no longer A1.30 (RUN), A2.30 (RUN)
- net SCL: now also J3.5 (SCL)
- net SDA: now also J3.6 (Pin_6)
- net SLAVEPWR: now also R1.1, J1.14 (Pin_14), J1.7 (Pin_7), R10.1, R11.1, R12.1, R9.1; no longer R1.2, R2.1
- net T_CLK: now reaches A2.14 (GPIO10)
- net T_CLK: now also J1.5 (Pin_5)
- net T_MOSI: now reaches A2.15 (GPIO11)
- net T_MOSI: now also J1.3 (Pin_3)
- net T_MISO: now reaches A2.16 (GPIO12)
- net T_MISO: now also J1.2 (Pin_2)
- net T_CS: now reaches A2.17 (GPIO13)
- net T_CS: now also R6.2, J1.4 (Pin_4)
- net T_INT: now reaches A2.19 (GPIO14)
- net T_INT: now also J1.1 (Pin_1)
- net E3A: now reaches A2.20 (GPIO15)
- net E3A: now also EC5.A, R12.2
- net E2B: now reaches A2.32 (GPIO27_ADC1)
- net E2B: now also EC4.B, R9.2
- net E2A: now reaches A2.34 (GPIO28_ADC2)
- net E2A: now also EC4.A, R10.2
- net E1B: now reaches A2.4 (GPIO2)
- net E1B: now also R5.2, EC3.B
- net E1A: now reaches A2.5 (GPIO3)
- net E1A: now also R7.2, EC3.A
- net MASTERPWR: now reaches A1.36 (3V3)
- removed net Card_CS: A2.27 (GPIO21), R6.2
- net INT: no longer names the net of A2.9 (GPIO6)
- net INT: no longer R5.2
- net LITE renamed E3B
- net E3B: now also EC5.B, R11.2
- new net: D82.4 (DOUT), D83.2 (DIN)
- new net: D83.4 (DOUT), D84.2 (DIN)
- new net: D118.4 (DOUT), D119.2 (DIN)
- new net: D108.4 (DOUT), D109.2 (DIN)
- new net: D109.4 (DOUT), D110.2 (DIN)
- new net: D92.4 (DOUT), D93.2 (DIN)
- new net: D148.4 (DOUT), D149.2 (DIN)
- new net: D149.4 (DOUT), D150.2 (DIN)
- new net: D124.4 (DOUT), D125.2 (DIN)
- new net: D125.4 (DOUT), D126.2 (DIN)
- new net: D93.4 (DOUT), D94.2 (DIN)
- new net: D94.4 (DOUT), D95.2 (DIN)
- new net: D139.4 (DOUT), D140.2 (DIN)
- new net: D140.4 (DOUT), D141.2 (DIN)
- new net: A2.30 (RUN), D161.2 (A)
- new net: D151.4 (DOUT), D152.2 (DIN)
- new net: D152.4 (DOUT), D153.2 (DIN)
- new net: D158.2 (A), EC3.S1
- new net: D120.4 (DOUT), D121.2 (DIN)
- new net: D121.4 (DOUT), D122.2 (DIN)
- new net: D133.4 (DOUT), D134.2 (DIN)
- new net: D134.4 (DOUT), D135.2 (DIN)
- new net: D160.2 (A), EC5.S1
- new net: D128.4 (DOUT), D129.2 (DIN)
- new net: D129.4 (DOUT), D130.2 (DIN)
- new net: D102.4 (DOUT), D103.2 (DIN)
- new net: D103.4 (DOUT), D104.2 (DIN)
- new net: D76.4 (DOUT), D80.2 (DIN)
- new net: D86.4 (DOUT), D87.2 (DIN)
- new net: D87.4 (DOUT), D88.2 (DIN)
- new net: D95.4 (DOUT), D96.2 (DIN)
- new net: D96.4 (DOUT), D97.2 (DIN)
- new net: D126.4 (DOUT), D127.2 (DIN)
- new net: D89.4 (DOUT), D90.2 (DIN)
- new net: D90.4 (DOUT), D91.2 (DIN)
- new net: D100.4 (DOUT), D101.2 (DIN)
- new net: D101.4 (DOUT), D102.2 (DIN)
- new net: D136.4 (DOUT), D137.2 (DIN)
- new net: D137.4 (DOUT), D138.2 (DIN)
- new net: D81.4 (DOUT), D82.2 (DIN)
- new net: D135.4 (DOUT), D136.2 (DIN)
- new net: D98.4 (DOUT), D99.2 (DIN)
- new net: D100.2 (DIN), D99.4 (DOUT)
- new net: D107.4 (DOUT), D108.2 (DIN)
- new net: D130.4 (DOUT), D131.2 (DIN)
- new net: D131.4 (DOUT), D132.2 (DIN)
- new net: D159.2 (A), EC4.S1
- new net: D150.4 (DOUT), D151.2 (DIN)
- new net: D80.4 (DOUT), D81.2 (DIN)
- new net: D141.4 (DOUT), D142.2 (DIN)
- new net: D110.4 (DOUT), D111.2 (DIN)
- new net: D106.4 (DOUT), D107.2 (DIN)
- new net: D114.4 (DOUT), D115.2 (DIN)
- new net: D115.4 (DOUT), D116.2 (DIN)
- new net: D122.4 (DOUT), D123.2 (DIN)
- new net: D117.4 (DOUT), D118.2 (DIN)
- new net: D153.4 (DOUT), D154.2 (DIN)
- new net: D97.4 (DOUT), D98.2 (DIN)
- new net: D142.4 (DOUT), D143.2 (DIN)
- new net: D138.4 (DOUT), D139.2 (DIN)
- new net: D112.4 (DOUT), D113.2 (DIN)
- new net: D113.4 (DOUT), D114.2 (DIN)
- new net: D85.4 (DOUT), D86.2 (DIN)
- new net: D123.4 (DOUT), D124.2 (DIN)
- new net: J1.11 (Pin_11), LEDDEBUG1.2, R1.2
- new net: D146.4 (DOUT), D147.2 (DIN)
- new net: D147.4 (DOUT), D148.2 (DIN)
- new net: D104.4 (DOUT), D105.2 (DIN)
- new net: D143.4 (DOUT), D144.2 (DIN)
- new net: D88.4 (DOUT), D89.2 (DIN)
- new net: D84.4 (DOUT), D85.2 (DIN)
- new net: D116.4 (DOUT), D117.2 (DIN)
- new net: D144.4 (DOUT), D145.2 (DIN)
- new net: D111.4 (DOUT), D112.2 (DIN)
- new net: D154.4 (DOUT), D155.2 (DIN)
- new net: D155.4 (DOUT), D156.2 (DIN)
- new net: A1.30 (RUN), D157.2 (A)
- new net: D127.4 (DOUT), D128.2 (DIN)
- new net LED1: D91.4 (DOUT), D92.2 (DIN)
- new net LED2: D105.4 (DOUT), D106.2 (DIN)
- new net LED3: D119.4 (DOUT), D120.2 (DIN)
- new net LED4: D132.4 (DOUT), D133.2 (DIN)
- new net LED5: D145.4 (DOUT), D146.2 (DIN)
- new net LEDData: A2.29 (GPIO22), D76.2 (DIN)
- new net LEDPWR: D100.3 (VDD), D101.3 (VDD), D102.3 (VDD), D103.3 (VDD), D104.3 (VDD), D105.3 (VDD), D106.3 (VDD), D107.3 (VDD), D108.3 (VDD), D109.3 (VDD), D110.3 (VDD), D111.3 (VDD), D112.3 (VDD), D113.3 (VDD), D114.3 (VDD), D115.3 (VDD), D116.3 (VDD), D117.3 (VDD), D118.3 (VDD), D119.3 (VDD), D120.3 (VDD), D121.3 (VDD), D122.3 (VDD), D123.3 (VDD), D124.3 (VDD), D125.3 (VDD), D126.3 (VDD), D127.3 (VDD), D128.3 (VDD), D129.3 (VDD), D130.3 (VDD), D131.3 (VDD), D132.3 (VDD), D133.3 (VDD), D134.3 (VDD), D135.3 (VDD), D136.3 (VDD), D137.3 (VDD), D138.3 (VDD), D139.3 (VDD), D140.3 (VDD), D141.3 (VDD), D142.3 (VDD), D143.3 (VDD), D144.3 (VDD), D145.3 (VDD), D146.3 (VDD), D147.3 (VDD), D148.3 (VDD), D149.3 (VDD), D150.3 (VDD), D151.3 (VDD), D152.3 (VDD), D153.3 (VDD), D154.3 (VDD), D155.3 (VDD), D156.3 (VDD), D76.3 (VDD), D80.3 (VDD), D81.3 (VDD), D82.3 (VDD), D83.3 (VDD), D84.3 (VDD), D85.3 (VDD), D86.3 (VDD), D87.3 (VDD), D88.3 (VDD), D89.3 (VDD), D90.3 (VDD), D91.3 (VDD), D92.3 (VDD), D93.3 (VDD), D94.3 (VDD), D95.3 (VDD), D96.3 (VDD), D97.3 (VDD), D98.3 (VDD), D99.3 (VDD), J5.2 (Pin_2)
- new net V+: J3.4 (Pin_4), J4.2 (Pin_2)
- no-connect marks 1 -> 36

Commit message: Finalized PCB files
Parts:
- added C1, C2: 10uF, Capacitor_SMD:C_1206_3216Metric_Pad1.33x1.80mm_HandSolder, symbol Device:C
- added C10, C11, C12, C3, C4, C5, C6, C7, C8, C9: 100nF, Capacitor_SMD:C_0805_2012Metric_Pad1.18x1.45mm_HandSolder, symbol Device:C
Connections:
- net GND: now also C1.1, C10.2, C11.2, C12.1, C2.2, C3.2, C4.2, C5.2, C6.2, C7.2, C8.2, C9.2
- net LEDPWR: now also C1.2, C10.1, C11.1, C2.1, C3.1, C4.1, C5.1, C6.1, C7.1, C8.1, C9.1
- net SLAVEPWR: now also C12.2
